File: 112.kicad_pcb (KiCad board)
At the start: 2 copper layers, 56.1 x 100.6 mm, 50 parts, among them J1 Conn_01x04, Q1 2N7000, Q2 2N7000, Q3 2N7000, Q4 2N7000, Q5 2N7000, Q6 2N7000, SW1 SW_DIP_x01, SW2 Rotary_Encoder_Switch, U1 STM32F103C8Tx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

Commit message: Add the work-in-progress version for future releases
Parts:
- added R26: 10k, Resistor_SMD:R_0805_2012Metric_Pad1.20x1.40mm_HandSolder, F.Cu at (59.9, 65.1)
- Q1, Q2, Q3, Q4, Q5, Q6: value 2N7000 -> 2N7002
- moved SW2 8.20 mm to (78.9, 66.1)
- moved R17 2.98 mm to (111.5, 112.3)
- moved R2 2.81 mm to (111.5, 101.8)
- moved R12 2.66 mm to (111.5, 124.8)
- moved R18 2.49 mm to (111.5, 135.3)
- moved R7 2.39 mm to (111.5, 91.6)
- moved R13 2.33 mm to (111.5, 145.8)
- moved R11 2.21 mm to (111.5, 143.8)
- moved R8 2.15 mm to (111.5, 93.6)
- moved R16 2.05 mm to (111.5, 133.3)
- moved R10 1.88 mm to (111.5, 122.8)
- moved R3 1.73 mm to (111.5, 103.8)
- moved R19 1.56 mm to (111.5, 114.3)
- moved R4 1.55 mm to (104.7, 102.8)
- moved R21 1.54 mm to (104.7, 113.3)
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Connections:
- Q1 pad 1: GND -> Net-(Q1-Pad1)
- Q1 pad 2: Net-(Q1-Pad2) -> GND
- Q2 pad 1: GND -> Net-(Q2-Pad1)
- Q2 pad 2: Net-(Q2-Pad2) -> GND
- Q3 pad 1: GND -> Net-(Q3-Pad1)
- Q3 pad 2: Net-(Q3-Pad2) -> GND
- Q4 pad 1: GND -> Net-(Q4-Pad1)
- Q4 pad 2: Net-(Q4-Pad2) -> GND
- Q5 pad 1: GND -> Net-(Q5-Pad1)
- Q5 pad 2: Net-(Q5-Pad2) -> GND
- Q6 pad 1: GND -> Net-(Q6-Pad1)
- Q6 pad 2: Net-(Q6-Pad2) -> GND
- R10 pad 1: Net-(Q3-Pad2) -> Net-(Q3-Pad1)
- R11 pad 1: Net-(Q1-Pad2) -> Net-(Q1-Pad1)
- R12 pad 2: Net-(Q3-Pad2) -> Net-(Q3-Pad1)
- R13 pad 2: Net-(Q1-Pad2) -> Net-(Q1-Pad1)
- R16 pad 1: Net-(Q2-Pad2) -> Net-(Q2-Pad1)
- R17 pad 1: Net-(Q4-Pad2) -> Net-(Q4-Pad1)
- R18 pad 2: Net-(Q2-Pad2) -> Net-(Q2-Pad1)
- R19 pad 2: Net-(Q4-Pad2) -> Net-(Q4-Pad1)
- R2 pad 1: Net-(Q5-Pad2) -> Net-(Q5-Pad1)
- R22 pad 1: +3V3 -> ENC_CLK
- R22 pad 2: ENC_CLK -> +3V3
- R23 pad 1: +3V3 -> ENC_DT
- R23 pad 2: ENC_DT -> +3V3
- R3 pad 2: Net-(Q5-Pad2) -> Net-(Q5-Pad1)
- R7 pad 1: Net-(Q6-Pad2) -> Net-(Q6-Pad1)
- R8 pad 2: Net-(Q6-Pad2) -> Net-(Q6-Pad1)
- SW2 pad S2: GND -> +3V3
- U1 pad 10: Net-(U1-Pad10) -> unconnected-(U1-Pad10)
- U1 pad 11: Net-(U1-Pad11) -> unconnected-(U1-Pad11)
- U1 pad 12: Net-(U1-Pad12) -> unconnected-(U1-Pad12)
- U1 pad 13: Net-(U1-Pad13) -> unconnected-(U1-Pad13)
- U1 pad 14: Net-(U1-Pad14) -> unconnected-(U1-Pad14)
- U1 pad 15: Net-(U1-Pad15) -> unconnected-(U1-Pad15)
- U1 pad 16: Net-(U1-Pad16) -> unconnected-(U1-Pad16)
- U1 pad 17: Net-(U1-Pad17) -> unconnected-(U1-Pad17)
- U1 pad 18: Net-(U1-Pad18) -> unconnected-(U1-Pad18)
- U1 pad 19: Net-(U1-Pad19) -> unconnected-(U1-Pad19)
- U1 pad 2: Net-(U1-Pad2) -> unconnected-(U1-Pad2)
- U1 pad 21: SCL -> unconnected-(U1-Pad21)
- U1 pad 22: Net-(U1-Pad22) -> unconnected-(U1-Pad22)
- U1 pad 25: Net-(U1-Pad25) -> unconnected-(U1-Pad25)
- U1 pad 26: Net-(U1-Pad26) -> unconnected-(U1-Pad26)
- U1 pad 3: Net-(U1-Pad3) -> unconnected-(U1-Pad3)
- U1 pad 34: Net-(U1-Pad34) -> unconnected-(U1-Pad34)
- U1 pad 37: Net-(U1-Pad37) -> unconnected-(U1-Pad37)
- U1 pad 4: Net-(U1-Pad4) -> unconnected-(U1-Pad4)
- U1 pad 42: Net-(U1-Pad42) -> unconnected-(U1-Pad42)
- U1 pad 43: Net-(U1-Pad43) -> unconnected-(U1-Pad43)
- U1 pad 45: Net-(U1-Pad45) -> DSP_SCL
- U1 pad 46: SDA -> DSP_SDA
- U1 pad 5: Net-(U1-Pad5) -> unconnected-(U1-Pad5)
- U1 pad 6: Net-(U1-Pad6) -> unconnected-(U1-Pad6)
- U4 pad 3: SDA -> DSP_SDA
- U4 pad 4: SCL -> DSP_SCL
Routing:
- net GND: track 260.4 -> 129.4 mm, vias 6 -> 4
- net +3V3: track 203.6 -> 112.7 mm, vias 4 -> 5
- net SDA: track 44.8 -> 0.00 mm, vias 2 -> 0
- net DSP_SDA: track 0.00 -> 44.8 mm, vias 0 -> 2
- net S4: track 81.8 -> 41.0 mm
- net S5: track 71.2 -> 30.4 mm
- net S3: track 92.1 -> 51.8 mm
- net S2: track 102.8 -> 62.6 mm
- net S6: track 60.5 -> 20.5 mm
- net S1: track 119.1 -> 80.7 mm
- net CONN+: track 32.9 -> 23.5 mm
- net Net-(Q4-Pad2): track 6.22 -> 0.00 mm
- net Net-(Q5-Pad2): track 6.11 -> 0.00 mm
- net Net-(Q1-Pad2): track 6.01 -> 0.00 mm
- net Net-(Q6-Pad2): track 6.01 -> 0.00 mm
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- removed copper zone on B.Cu, net GND
- removed copper zone on F.Cu, net GND
Other:
- net class Default removed

Commit message: Update PCB layout
Parts:
- moved R26 4.75 mm to (64.7, 65.1), turned to -90 degrees
Changed lines of the file:
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@@
   )
   (footprint "Resistor_SMD:R_0805_2012Metric_Pad1.20x1.40mm_HandSolder" (layer "F.Cu")
-    (at 59.901 65.087 180)
+    (at 64.651 65.087 -90)
     (descr "Resistor SMD 0805 (2012 Metric), square (rectangular) end terminal, IPC_7351 nominal with elongated pad for handsoldering. (Body size source: IPC-SM-782 page 72, https://www.pcb-3d.com/wordpress/wp-content/uploads/ipc-sm-782a_amendment_1_and_2.pdf), generated with kicad-footprint-generator")
     (tags "resistor handsolder")
@@
     (property "Sheetname" "")
     (attr smd)
-    (fp_text reference "R26" (at 0 -1.65) (layer "F.SilkS")
+    (fp_text reference "R26" (at 0 -1.65 -270) (layer "F.SilkS")
       (effects (font (size 1 1) (thickness 0.15)))
     )
-    (fp_text value "10k" (at 0 1.65) (layer "F.Fab")
+    (fp_text value "10k" (at 0 1.65 -270) (layer "F.Fab")
       (effects (font (size 1 1) (thickness 0.15)))
     )
-    (fp_text user "${REFERENCE}" (at 0 0) (layer "F.Fab")
+    (fp_text user "${REFERENCE}" (at 0 0 -270) (layer "F.Fab")
       (effects (font (size 0.5 0.5) (thickness 0.08)))
     )
@@
     (fp_line (start 1 -0.625) (end 1 0.625) (layer "F.Fab") (width 0.1))
     (fp_line (start -1 0.625) (end -1 -0.625) (layer "F.Fab") (width 0.1))
-    (pad "1" smd roundrect locked (at -1 0 180) (size 1.2 1.4) (layers "F.Cu" "F.Paste" "F.Mask") (roundrect_rratio 0.208333)
+    (pad "1" smd roundrect locked (at -1 0 270) (size 1.2 1.4) (layers "F.Cu" "F.Paste" "F.Mask") (roundrect_rratio 0.208333)
       (net 3 "GND") (pintype "passive"))
-    (pad "2" smd roundrect locked (at 1 0 180) (size 1.2 1.4) (layers "F.Cu" "F.Paste" "F.Mask") (roundrect_rratio 0.208333)
+    (pad "2" smd roundrect locked (at 1 0 270) (size 1.2 1.4) (layers "F.Cu" "F.Paste" "F.Mask") (roundrect_rratio 0.208333)
       (net 27 "ENC_BTN") (pintype "passive"))
     (model "${KICAD6_3DMODEL_DIR}/Resistor_SMD.3dshapes/R_0805_2012Metric.wrl"
